File: Hardware/Water_Quality_Measuring_System.kicad_pcb (KiCad board)
At the start: 2 copper layers, 85.2 x 51.7 mm, 58 parts, among them IC1 LP2992IM5-3.3, IC2 LP2992IM5-3.3, IC3 LP2992IM5-3.3, J1 USB_C_Receptacle, Q1 S8050, Q2 S8050, Q3 S8050, Q4 S8050, U1 ESP32-PICO-D4, U2 CP2102N-Axx-xQFN28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

Commit message: First Commit
Parts:
- moved R18 2.52 mm to (129.1, 37.4), turned to 0 degrees
- moved R19 2.50 mm to (129.1, 34.9), turned to 0 degrees
- moved C4 0.07 mm to (152.0, 30.1)
Connections:
- U4 pad 18: /LCD_CS -> GND
Routing:
- net /SENSOR_SCL: track 0.00 -> 49.1 mm, vias 0 -> 2
- net /SENSOR_SDA: track 0.00 -> 41.3 mm, vias 0 -> 2
- net /LCD_DC: track 0.00 -> 28.1 mm
- net /LCD_RES: track 0.00 -> 27.1 mm
- net /SENSOR_VCC: track 12.7 -> 33.5 mm, vias 0 -> 3
- net /LCD_MOSI: track 0.00 -> 19.8 mm
- net /LCD_CLK: track 0.00 -> 18.7 mm, vias 0 -> 2
- net /U0TXD: track 0.00 -> 10.4 mm, vias 0 -> 2
- net /U0RXD: track 0.00 -> 10.4 mm, vias 0 -> 2
- net +3.3V: track 28.7 -> 36.4 mm
- net +5V: track 38.6 -> 45.7 mm
- net /EN: track 0.00 -> 4.50 mm
- net Net-(U2-~{RST}): track 0.00 -> 1.81 mm

Commit message: Finished PCB Layout
Parts:
- added U5: TP4055-42-SOT25-R, kicad_lceda:SOT-23-5_L2.9-W1.6-P0.95-LS2.8-BL, F.Cu at (114.2, 104.6)
- added U6: EC190707, kicad_lceda:EC190707_STD, F.Cu at (109.8, 104.9)
- AE1: footprint RF_Antenna:Texas_SWRA117D_2.4GHz_Right -> RF_Antenna:Johanson_2450AT43F0100
- moved AE1 4.34 mm to (146.2, 76.0)
Connections:
- U1 pad 18: unconnected-(U1-IO12-Pad18) -> /KEY_D
- U1 pad 28: unconnected-(U1-SD2/IO9-Pad28) -> /KEY_E
- U1 pad 29: unconnected-(U1-SD3/IO10-Pad29) -> /KEY_U
- U1 pad 38: unconnected-(U1-IO19-Pad38) -> /KEY_L
- U1 pad 42: unconnected-(U1-IO21-Pad42) -> /KEY_R
Routing:
- net +3.3V: track 36.4 -> 115.6 mm, vias 0 -> 8
- net /KEY_R: track 1.89 -> 48.9 mm, vias 0 -> 2
- net +5V: track 45.7 -> 91.4 mm, vias 4 -> 8
- net /LCD_VCC: track 18.2 -> 62.6 mm, vias 1 -> 3
- net /KEY_L: track 1.92 -> 42.4 mm, vias 0 -> 2
- net Net-(AE1-A): track 0.00 -> 32.9 mm, vias 0 -> 2
- net /KEY_D: track 2.12 -> 27.9 mm, vias 0 -> 2
- net /KEY_U: track 2.08 -> 27.1 mm, vias 0 -> 2
- net /KEY_E: track 2.15 -> 23.9 mm, vias 0 -> 2
- net /LCD_BLK: track 0.00 -> 19.5 mm, vias 0 -> 1
- net /GPIO_0: track 0.00 -> 16.5 mm, vias 0 -> 2
- net Net-(D2-K): track 3.49 -> 18.0 mm, vias 0 -> 2
- net /EN: track 4.50 -> 16.7 mm, vias 0 -> 2
- net Net-(IC2-BYPASS): track 0.00 -> 1.76 mm
- net /SD_CS: track 31.5 -> 32.5 mm
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- added copper zone on B.Cu, net GND
- added copper zone on F.Cu, net GND
Other:
- outline, holes or cut-outs redrawn

Commit message: Finished Main Board PCB
Parts:
- added C16: 10uF, Capacitor_SMD:C_0603_1608Metric, F.Cu at (122.9, 103.1)
- added C17: 1uF, Capacitor_SMD:C_0603_1608Metric, F.Cu at (122.9, 105.6)
- added C18: 10uF, Capacitor_SMD:C_0603_1608Metric, F.Cu at (122.9, 108.1)
- added D4: LED, LED_SMD:LED_0603_1608Metric, F.Cu at (126.9, 110.5)
- added D5: 1N5819WS, Diode_SMD:D_SOD-323, F.Cu at (127.1, 107.7)
- added R26: 10K, Resistor_SMD:R_0603_1608Metric, F.Cu at (122.9, 110.6)
- added R27: 1.66K, Resistor_SMD:R_0603_1608Metric, F.Cu at (122.9, 113.2)
- added SW1: Power, Button_Switch_SMD:SW_SPST_B3U-1000P, F.Cu at (127.8, 104.0)
Connections:
- C10 pad 1: +5V -> /BAT_OUT
- C13 pad 1: +5V -> /BAT_OUT
- C7 pad 1: +5V -> /BAT_OUT
- IC1 pad 1: +5V -> /BAT_OUT
- IC1 pad 3: +5V -> /BAT_OUT
- IC2 pad 1: +5V -> /BAT_OUT
- IC2 pad 3: +5V -> /BAT_OUT
- IC3 pad 1: +5V -> /BAT_OUT
- IC3 pad 3: +5V -> /BAT_OUT
- U5 pad 1: unconnected-(U5-CHRG-Pad1) -> Net-(D4-K)
- U5 pad 2: unconnected-(U5-GND-Pad2) -> GND
- U5 pad 3: unconnected-(U5-BAT-Pad3) -> /BAT+
- U5 pad 4: unconnected-(U5-VCC-Pad4) -> +5V
- U5 pad 5: unconnected-(U5-PROG-Pad5) -> Net-(U5-PROG)
- U6 pad 1: unconnected-(U6-OUT-Pad1) -> /BAT_OUT
- U6 pad 2: unconnected-(U6-GND-Pad2) -> GND
- U6 pad 3: unconnected-(U6-KEY-Pad3) -> Net-(D5-A)
- U6 pad 5: unconnected-(U6-VDD-Pad5) -> /BAT+
