File: Hardware/Water_Quality_Measuring_System.kicad_sch (KiCad schematic)
At the start: 58 parts, among them IC1 LP2992IM5-3.3, J1 USB_C_Receptacle, Q1 S8050, Q2 S8050, Q3 S8050, Q4 S8050, U1 ESP32-PICO-D4, U2 CP2102N-Axx-xQFN28, U3 五向开关

Commit message: First Commit
Connections:
- net LCD_CS is gone; now on net GND: U4.18 (CS)
Changed lines of the file:
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@@
+    )
+  )
+  (symbol (lib_id "power:GND") (at 152.4 244.856 90) (unit 1)
+    (in_bom yes) (on_board yes) (dnp no) (fields_autoplaced)
+    (property "Reference" "#PWR021" (at 158.75 244.856 0)
+      (effects (font (size 1.27 1.27)) hide)
+    )
+    (property "Value" "GND" (at 156.464 244.856 90)
+      (effects (font (size 1.27 1.27)) (justify right))
+    )
+    (property "Footprint" "" (at 152.4 244.856 0)
+      (effects (font (size 1.27 1.27)) hide)
+    )
+    (property "Datasheet" "" (at 152.4 244.856 0)
+      (effects (font (size 1.27 1.27)) hide)
+    )
+    (pin "1")
+    (instances
+      (project "DRV8313_Dev_Board"
+        (path "/68230e14-bdbb-403c-82a7-6b8a172d069e"
+          (reference "#PWR021") (unit 1)
+        )
+      )
+      (project "Water_Quality_Measuring_System"
+        (path "/7b51d846-b8d6-4f13-b74f-f62264261045"
+          (reference "#PWR022") (unit 1)
+        )
+      )
     )
   )

Commit message: Finished PCB Layout
Parts:
- added U5: TP4055-42-SOT25-R, kicad_lceda:SOT-23-5_L2.9-W1.6-P0.95-LS2.8-BL, symbol kicad_lceda:TP4055-42-SOT25-R
- added U6: EC190707, kicad_lceda:EC190707_STD, symbol kicad_lceda:EC190707
- AE1: footprint RF_Antenna:Texas_SWRA117D_2.4GHz_Right -> RF_Antenna:Johanson_2450AT43F0100
Connections:
- net KEY_D: now also U1.18 (IO12)
- net KEY_E: now also U1.28 (SD2/IO9)
- net KEY_L: now also U1.38 (IO19)
- net KEY_R: now also U1.42 (IO21)
- net KEY_U: now also U1.29 (SD3/IO10)
Changed lines of the file:
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@@
-    (stroke (width 0) (type default))
-  )
-  (wire (pts (xy 136.144 90.424) (xy 121.666 90.424))
     (stroke (width 0) (type default))
   )
@@
     (stroke (width 0) (type default))
   )
+  (wire (pts (xy 121.666 103.124) (xy 136.398 103.124))
+    (stroke (width 0) (type default))
+  )
   (wire (pts (xy 282.194 146.812) (xy 289.052 146.812))
     (stroke (width 0) (type default))
   )
+  (wire (pts (xy 121.666 87.884) (xy 136.144 87.884))
+    (stroke (width 0) (type default))
+  )
   (wire (pts (xy 83.566 53.086) (xy 83.566 53.848))
     (stroke (width 0) (type default))
@@
     (stroke (width 0) (type default))
   )
-  (wire (pts (xy 136.144 98.044) (xy 121.666 98.044))
+  (wire (pts (xy 136.398 98.044) (xy 121.666 98.044))
     (stroke (width 0) (type default))
   )
@@
     (stroke (width 0) (type default))
   )
+  (wire (pts (xy 121.666 90.424) (xy 136.398 90.424))
+    (stroke (width 0) (type default))
+  )
   (wire (pts (xy 234.188 217.932) (xy 249.174 217.932))
     (stroke (width 0) (type default))
@@
     (stroke (width 0) (type default))
   )
+  (wire (pts (xy 121.666 85.344) (xy 136.144 85.344))
+    (stroke (width 0) (type default))
+  )
   (wire (pts (xy 335.026 200.914) (xy 343.408 200.914))
     (stroke (width 0) (type default))
@@
     (stroke (width 0) (type default))
   )
+  (wire (pts (xy 121.666 100.584) (xy 136.398 100.584))
+    (stroke (width 0) (type default))
+  )
   (wire (pts (xy 289.052 141.732) (xy 289.052 139.192))
     (stroke (width 0) (type default))
@@
     (stroke (width 0) (type default))
   )
-  (wire (pts (xy 136.144 92.964) (xy 121.666 92.964))
-    (stroke (width 0) (type default))
-  )
   (wire (pts (xy 145.288 234.696) (xy 145.288 237.236))
     (stroke (width 0) (type default))
@@
     (stroke (width 0) (type default))
   )
+  (wire (pts (xy 121.666 82.804) (xy 136.144 82.804))
+    (stroke (width 0) (type default))
+  )
   (wire (pts (xy 234.696 27.686) (xy 237.49 27.686))
     (stroke (width 0) (type default))
   )
+  (wire (pts (xy 121.666 95.504) (xy 136.398 95.504))
+    (stroke (width 0) (type default))
+  )
   (wire (pts (xy 253.238 252.476) (xy 253.238 252.73))
     (stroke (width 0) (type default))
   )
+  (wire (pts (xy 121.666 92.964) (xy 136.398 92.964))
+    (stroke (width 0) (type default))
+  )
   (wire (pts (xy 188.722 195.58) (xy 180.34 195.58))
     (stroke (width 0) (type default))
@@
     (stroke (width 0) (type default))
   )
-  (wire (pts (xy 136.144 95.504) (xy 121.666 95.504))
-    (stroke (width 0) (type default))
-  )
   (wire (pts (xy 330.708 135.89) (xy 345.694 135.89))
     (stroke (width 0) (type default))
@@
     (effects (font (size 1.27 1.27)) (justify right bottom))
   )
-  (label "SD_CS" (at 136.144 95.504 180) (fields_autoplaced)
+  (label "SD_CS" (at 136.398 95.504 180) (fields_autoplaced)
     (effects (font (size 1.27 1.27)) (justify right bottom))
   )
@@
     (effects (font (size 1.27 1.27)) (justify right bottom))
   )
+  (label "KEY_U" (at 136.144 85.344 180) (fields_autoplaced)
+    (effects (font (size 1.27 1.27)) (justify right bottom))
+  )
   (label "SENSOR_VP" (at 67.31 67.564 0) (fields_autoplaced)
     (effects (font (size 1.27 1.27)) (justify left bottom))
@@
     (effects (font (size 1.27 1.27)) (justify right bottom))
   )
-  (label "SD_MOSI" (at 136.144 90.424 180) (fields_autoplaced)
+  (label "SD_MOSI" (at 136.398 90.424 180) (fields_autoplaced)
     (effects (font (size 1.27 1.27)) (justify right bottom))
   )
@@
     (effects (font (size 1.27 1.27)) (justify left bottom))
   )
+  (label "KEY_R" (at 136.398 103.124 180) (fields_autoplaced)
+    (effects (font (size 1.27 1.27)) (justify right bottom))
+  )
   (label "DTR" (at 331.216 54.102 180) (fields_autoplaced)
     (effects (font (size 1.27 1.27)) (justify right bottom))
   )
-  (label "SD_CLK" (at 136.144 92.964 180) (fields_autoplaced)
+  (label "SD_CLK" (at 136.398 92.964 180) (fields_autoplaced)
     (effects (font (size 1.27 1.27)) (justify right bottom))
   )
@@
     (effects (font (size 1.27 1.27)) (justify left bottom))
   )
+  (label "KEY_L" (at 136.398 100.584 180) (fields_autoplaced)
+    (effects (font (size 1.27 1.27)) (justify right bottom))
+  )
   (label "KEY_U" (at 335.026 195.834 0) (fields_autoplaced)
     (effects (font (size 1.27 1.27)) (justify left bottom))
@@
     (effects (font (size 1.27 1.27)) (justify right bottom))
   )
+  (label "KEY_D" (at 136.144 87.884 180) (fields_autoplaced)
+    (effects (font (size 1.27 1.27)) (justify right bottom))
+  )
   (label "FLASH_SD3" (at 67.31 103.124 0) (fields_autoplaced)
     (effects (font (size 1.27 1.27)) (justify left bottom))
@@
     (effects (font (size 1.27 1.27)) (justify left bottom))
   )
-  (label "LCD_CLK" (at 136.144 98.044 180) (fields_autoplaced)
+  (label "LCD_CLK" (at 136.398 98.044 180) (fields_autoplaced)
     (effects (font (size 1.27 1.27)) (justify right bottom))
   )
@@
   (label "EN" (at 291.338 43.18 0) (fields_autoplaced)
     (effects (font (size 1.27 1.27)) (justify left bottom))
+  )
+  (label "KEY_E" (at 136.144 82.804 180) (fields_autoplaced)
+    (effects (font (size 1.27 1.27)) (justify right bottom))
   )
   (label "LCD_MOSI" (at 152.4 252.476 180) (fields_autoplaced)
@@
     )
   )
+  (symbol (lib_id "kicad_lceda:TP4055-42-SOT25-R") (at 176.276 153.924 0) (unit 1)
+    (in_bom yes) (on_board yes) (dnp no) (fields_autoplaced)
+    (property "Reference" "U5" (at 176.276 143.51 0)
+      (effects (font (size 1.27 1.27)))
+    )
+    (property "Value" "TP4055-42-SOT25-R" (at 176.276 146.05 0)
+      (effects (font (size 1.27 1.27)))
+    )
+    (property "Footprint" "kicad_lceda:SOT-23-5_L2.9-W1.6-P0.95-LS2.8-BL" (at 176.276 151.257 0)
+      (effects (font (size 1.27 1.27)) hide)
+    )
+    (property "Datasheet" "" (at 176.276 156.337 0)
+      (effects (font (size 1.27 1.27)) hide)
+    )
+    (property "SuppliersPartNumber" "C2925180" (at 176.276 161.417 0)
+      (effects (font (size 1.27 1.27)) hide)
+    )
+    (property "uuid" "std:6f29a4b961dc4e909225a40f3dd98aae" (at 176.276 161.417 0)
+      (effects (font (size 1.27 1.27)) hide)
+    )
+    (pin "1")
+    (pin "2")
+    (pin "3")
+    (pin "4")
+    (pin "5")
+    (instances
+      (project "Water_Quality_Measuring_System"
+        (path "/7b51d846-b8d6-4f13-b74f-f62264261045"
+          (reference "U5") (unit 1)
+        )
+      )
+    )
+  )
   (symbol (lib_id "SamacSys_Parts:TCS34725") (at 239.522 189.484 0) (unit 1)
     (in_bom yes) (on_board yes) (dnp no) (fields_autoplaced)
@@
       (effects (font (size 1.27 1.27)) (justify left))
     )
-    (property "Footprint" "RF_Antenna:Texas_SWRA117D_2.4GHz_Right" (at 134.112 50.8 0)
+    (property "Footprint" "RF_Antenna:Johanson_2450AT43F0100" (at 134.112 50.8 0)
       (effects (font (size 1.27 1.27)) hide)
     )
@@
         )
       )
+    )
+  )
+  (symbol (lib_id "kicad_lceda:EC190707") (at 169.418 127 0) (unit 1)
+    (in_bom yes) (on_board yes) (dnp no) (fields_autoplaced)
+    (property "Reference" "U6" (at 175.768 106.68 0)
+      (effects (font (size 1.27 1.27)))
+    )
+    (property "Value" "EC190707" (at 175.768 109.22 0)
+      (effects (font (size 1.27 1.27)))
+    )
+    (property "Footprint" "kicad_lceda:EC190707_STD" (at 169.418 114.2238 0)
+      (effects (font (size 1.27 1.27)) hide)
+    )
+    (property "Datasheet" "" (at 169.418 119.3038 0)
+      (effects (font (size 1.27 1.27)) hide)
+    )
+    (property "SuppliersPartNumber" "" (at 169.418 124.3838 0)
+      (effects (font (size 1.27 1.27)) hide)
+    )
+    (property "uuid" "std:2dd3d4a6db3b470aa9ff21f38ac65896" (at 169.418 124.3838 0)
+      (effects (font (size 1.27 1.27)) hide)
+    )
+    (pin "1")
+    (pin "2")
+    (pin "3")
+    (pin "4")
+    (pin "5")
+    (pin "6")
+    (instances
+      (project "Water_Quality_Measuring_System"
+        (path "/7b51d846-b8d6-4f13-b74f-f62264261045"
+          (reference "U6") (unit 1)
+        )
+      )

Commit message: Finished Main Board PCB
Parts:
- added C16, C18: 10uF, Capacitor_SMD:C_0603_1608Metric, symbol Device:C
- added C17: 1uF, Capacitor_SMD:C_0603_1608Metric, symbol Device:C
- added D4: LED, LED_SMD:LED_0603_1608Metric, symbol Device:LED
- added D5: 1N5819WS, Diode_SMD:D_SOD-323, symbol Diode:1N5819WS
- added R26: 10K, Resistor_SMD:R_0603_1608Metric, symbol Device:R
- added R27: 1.66K, Resistor_SMD:R_0603_1608Metric, symbol Device:R
- added SW1: Power, Button_Switch_SMD:SW_SPST_B3U-1000P, symbol Switch:SW_Push
Connections:
- net +5V: now also U5.4 (VCC), C17.2, R26.1; no longer C2.1, C2.1, C2.1, IC1.1 (IN), IC1.1 (IN), IC1.1 (IN), IC1.3 (ON/~{OFF}), IC1.3 (ON/~{OFF}), IC1.3 (ON/~{OFF})
- net GND: now also U5.2 (GND), U6.2 (GND), C16.1, C17.1, C18.1, D5.1 (K), R27.2, SW1.1
- net at U5.1 (CHRG): now also D4.1 (K)
- net BAT+: now reaches U5.3 (BAT)
- net BAT+: now also U6.5 (VDD), C16.2, C18.2
- net at U5.5 (PROG): now also R27.1
- net BAT_OUT: now reaches U6.1 (OUT)
- net BAT_OUT: now also C2.1, C2.1, C2.1, IC1.1 (IN), IC1.1 (IN), IC1.1 (IN), IC1.3 (ON/~{OFF}), IC1.3 (ON/~{OFF}), IC1.3 (ON/~{OFF})
- net at U6.3 (KEY): now also D5.2 (A), SW1.2
- new net: D4.2 (A), R26.2
- no-connect marks 31 -> 33
Other:
- moved on the sheet: AE1, C1, C2, C3, R1, U1, U5, U6
