File: Hardware/Main_Board/Main_Board.kicad_pcb (KiCad board)
At the start: 2 copper layers, 50 x 36.5 mm, 49 parts, among them IC1 LP2992IM5-3.3, IC2 LP2992IM5-3.3, IC3 LP2992IM5-3.3, J1 USB_C_Receptacle, J2 LCD&KEYS, J3 Sensor_Connector, Q1 S8050, Q2 S8050, U1 ESP32-PICO-D4, U2 CP2102N-Axx-xQFN28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

Commit message: Finished All PCB
Parts:
- added J4: BattaryPack_18650, Resistor_SMD:R_2816_7142Metric_Pad3.20x4.45mm_HandSolder, F.Cu at (63.7, 58.7)
- IC1, IC2, IC3: footprint SamacSys_Parts:SOT95P280X145-5N -> Library:SOT95P280X145-5N
- Q1, Q2: footprint SamacSys_Parts:SOT95P240X115-3N -> Library:SOT95P240X115-3N
- moved AE1 47.5 mm to (33.1, 59.6)
- moved R14 47.5 mm to (50.8, 57.6)
- moved U3 47.5 mm to (53.4, 57.8)
- moved C1 47.5 mm to (45.8, 49.6)
- moved C11 47.5 mm to (68.4, 54.5)
- moved C13 47.5 mm to (60.4, 52.2)
- moved C6 47.5 mm to (68.4, 48.7)
- moved C8 47.5 mm to (58.1, 48.7)
- moved C9 47.5 mm to (58.1, 54.5)
- moved D2 47.5 mm to (51.5, 60.6)
- moved H1 47.5 mm to (48.7, 30.7)
- moved H3 47.5 mm to (74.3, 56.5)
- moved IC1 47.5 mm to (57.8, 51.6)
- moved IC3 47.5 mm to (68.1, 51.6)
- moved R1 47.5 mm to (46.9, 50.6)
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Connections:
- J3 pad 2: /SENSOR_VCC -> /SENSOR_INT
- U1 pad 11: unconnected-(U1-IO35-Pad11) -> /SENSOR_INT
Routing:
- net +3.3V: track 12.4 -> 90.1 mm, vias 0 -> 10
- net /BAT_OUT: track 15.9 -> 63.7 mm, vias 0 -> 2
- net /BAT+: track 1.56 -> 49.2 mm, vias 0 -> 2
- net /SENSOR_VCC: track 1.68 -> 26.9 mm, vias 0 -> 2
- net +5V: track 25.6 -> 48.8 mm, vias 2 -> 4
- net /LCD_VCC: track 1.68 -> 15.3 mm
- net /SENSOR_INT: track 0.00 -> 10.9 mm, vias 0 -> 2
- net /KEY_L: track 30.7 -> 31.7 mm
- net /KEY_R: track 33.1 -> 34.1 mm
- net GND: vias 0 -> 38
- added copper zone on B.Cu, net GND
- added copper zone on F.Cu, net GND
Other:
- outline, holes or cut-outs redrawn
- board text added: "+"
- board text added: "0"
- board text added: "0 mm"
- board text added: "0.01 mm"
- board text added: "0.02"
- board text added: "0.035 mm"
- board text added: "1"
- board text added: "1.51 mm"
- board text added: "3.3"
- board text added: "4.5"
- board text added: "B.Cu"
- board text added: "B.Mask"
- board text added: "B.Paste"
- board text added: "B.Silkscreen"
- board text added: "BAT"
- board text added: "Bottom Silk Screen"
- board text added: "Bottom Solder Mask"
- board text added: "Bottom Solder Paste"
- board text added: "Epsilon R"
- board text added: "F.Cu"
- board text added: "F.Mask"
- board text added: "F.Paste"
- board text added: "F.Silkscreen"
- board text added: "FR4"
- board text added: "Loss Tangent"
- board text added: "Not specified"
- board text added: "Top Silk Screen"
- board text added: "Top Solder Mask"
- board text added: "Top Solder Paste"
- board text added: "copper"
- board text added: "core"
- board text added: "介质"
- board text added: "厚度 (mm)"
- board text added: "层名称"
- board text added: "材料"
- board text added: "类型"
- board text added: "颜色"
