File: Hardware/Main_Board/Main_Board.kicad_sch (KiCad schematic)
At the start: 49 parts, among them IC1 LP2992IM5-3.3, J1 USB_C_Receptacle, J2 LCD&KEYS, J3 Sensor_Connector, Q1 S8050, Q2 S8050, U1 ESP32-PICO-D4, U2 CP2102N-Axx-xQFN28, U5 TP4055-42-SOT25-R

Commit message: Finished All PCB
Parts:
- added J4: BattaryPack_18650, Resistor_SMD:R_2816_7142Metric_Pad3.20x4.45mm_HandSolder, symbol Connector:Conn_01x02_Socket
Connections:
- net BAT+: now also J4.1 (Pin_1)
- net GND: now also J4.2 (Pin_2)
- net SENSOR_VCC: no longer J3.2 (Pin_2)
- net SENSOR_INT: now reaches U1.11 (IO35)
- net SENSOR_INT: now also J3.2 (Pin_2)
Other:
- moved on the sheet: J2, J3
